File: 2_channel_relay_module_Replica/2_channel_relay_module/2_channel_relay_module.kicad_sch (KiCad schematic)
At the start: 25 parts, among them J1 Bornera, J2 Bornera, J3 Tiras de pines macho, J4 Tira de pines macho, K1 SONGLE_SRD_Form_C, K2 SONGLE_SRD_Form_C, Q1 S8050, Q2 S8050, U1 PC817, U2 PC817

Commit message: commit_02
Parts:
- D1, D2: Catalogo (none) -> https://www.microelectronicash.com/~microelect/detalle.php?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
- F1, F2, F3: footprint Fiducial:Fiducial_0.5mm_Dia_1mm_Outer -> Fiducial:Fiducial_0.5mm_Mask1.5mm
- IN1, IN2: Catalogo (none) -> http://www.microelectronicash.com/l-1206r--det--L-1206R
- J1, J2: Catalogo (none) -> https://electronica-jm.com/product/bornera-verde-3-pines/
- J3: footprint (none) -> Connector_PinHeader_2.54mm:PinHeader_1x03_P2.54mm_Vertical; Catalogo (none) -> http://www.microelectronicash.com/tp1x20-2-00--det--TP1X20-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
- J4: footprint (none) -> Connector_PinHeader_2.54mm:PinHeader_1x04_P2.54mm_Vertical; Catalogo (none) -> http://www.microelectronicash.com/tp1x20-2-00--det--TP1X20-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
- K1, K2: Catalogo (none) -> https://candy-ho.com/producto/modulo-rele-5v-simple-inverso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
- Q1, Q2: Catalogo (none) -> https://www.digikey.com/en/products/detail/micro-commercial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
- R1, R3: Catalogo (none) -> http://www.microelectronicash.com/r1206-1k--det--R1206-1K
- R2, R4: Catalogo (none) -> https://mvelectronica.com/producto/510-ohms-resistencia-smd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
- U1, U2: Catalogo (none) -> https://www.digikey.com/es/products/detail/sharp-socle-tech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
Connections:
- net at J2.1 (Pin_1): now also K2.3; no longer K2.4
- net at J2.3 (Pin_3): now also K2.4; no longer K2.3
- net at J1.1 (Pin_1): now also K1.3; no longer K1.4
- net at J1.3 (Pin_3): now also K1.4; no longer K1.3
Other:
- note added: "COM"
- note added: "NC"
- note added: "NO"
- note added: "Pin 1: RY-VCC (5V fuente adicional) Pin 2: VCC (5V) Pin 3: GND"
- note added: "Pin 1: VCC (5V) Pin 2: IN2 Pin 3: IN1 Pin 4: GND"
- note added: "Pines 1 y 2 van puenteados con un jumper, si se necesita conducir una gran potencia de carga, se puede quitar el jumper y conectar una fuente adicional de 5 V en RY-VCC para alimentar los relés."
